File: Ball Butler/ball_butler_circuit_diagram/ball_butler_circuit_diagram.kicad_sch (KiCad schematic)
At the start: 16 parts

Commit message: Update Ball Butler schematic
Connections:
- net at U?. (NC): now also U?. (VIN)
- new net: U?. (GND), U?. (GND) (x3)
- new net: M?. (C), U?. (VIN) (x4)
- new net: U?. (PIN), U?. (VIN)
- new net: M?. (PWR2), U?. (VIN)
- new net: U?. (NC), U?. (VIN) (x4)
Changed lines of the file:
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@@
       (reference "U?") (unit 1) (value "ODrive_S1") (footprint "")
+    )
+    (path "/f47f7cdf-3580-439c-86a6-80f9e434af39/10f59d9c-3790-448c-bf85-4703c260aa1f"
+      (reference "U?") (unit 1) (value "ball_reloader") (footprint "")
     )
     (path "/19948f7d-0628-4718-a282-ada50b0a9773"
@@
     (path "/f47f7cdf-3580-439c-86a6-80f9e434af39/20395ea7-59ae-452e-9250-0e0b18719f6f"
       (reference "U?") (unit 1) (value "can1_receiver") (footprint "")
-    )
-    (path "/f47f7cdf-3580-439c-86a6-80f9e434af39/24b6e83c-fa1f-4658-a814-2d4625a7322c"
-      (reference "U?") (unit 1) (value "store_throw_num") (footprint "")
     )
     (path "/3005be57-9842-4134-96d2-a3e5d7976d31"
@@
       (reference "U?") (unit 1) (value "Jetson") (footprint "")
     )
+    (path "/f47f7cdf-3580-439c-86a6-80f9e434af39/53aec20f-7713-41a6-b582-41eed197c871"
+      (reference "U?") (unit 1) (value "Yaw_Proprioception") (footprint "")
+    )
     (path "/8ed858a8-e638-495c-b31c-77c4342d4bce/5bb9813c-597e-4535-9c13-aa1ef03c8eb5"
       (reference "U?") (unit 1) (value "ODrive Pro 4") (footprint "")
-    )
-    (path "/f47f7cdf-3580-439c-86a6-80f9e434af39/5d3cd58b-8c1f-43a4-bfdd-2f8217b9e1ab"
-      (reference "U?") (unit 1) (value "ballistics_calculator") (footprint "")
     )
     (path "/f47f7cdf-3580-439c-86a6-80f9e434af39/61607c88-2168-4de3-ba26-a1c5c3e03fa5"
@@
       (reference "U?") (unit 1) (value "ODrive Pro 6") (footprint "")
     )
-    (path "/f47f7cdf-3580-439c-86a6-80f9e434af39/78cd3d64-8d8b-4280-a96d-a5b38f46313b"
-      (reference "U?") (unit 1) (value "can1_receiver") (footprint "")
+    (path "/f47f7cdf-3580-439c-86a6-80f9e434af39/733c6df0-59cf-4e7f-8850-809c638a8458"
+      (reference "U?") (unit 1) (value "proprioception_handler") (footprint "")
     )
     (path "/7c8e867e-26c4-4035-bf4a-5d705b8387f3"
       (reference "U?") (unit 1) (value "CAN_Transceiver") (footprint "")
-    )
-    (path "/f47f7cdf-3580-439c-86a6-80f9e434af39/82a2bb4f-00c5-49ad-971c-7b74231ecae0"
-      (reference "U?") (unit 1) (value "can1_transmitter") (footprint "")
-    )
-    (path "/f47f7cdf-3580-439c-86a6-80f9e434af39/976d4190-3ffb-4a7d-9f5d-de19a9216559"
-      (reference "U?") (unit 1) (value "IK_solver") (footprint "")
     )
     (path "/8ed858a8-e638-495c-b31c-77c4342d4bce/a103d190-b91c-4b7f-9aad-b47edf75f452"
@@
       (reference "U?") (unit 1) (value "ODrive Pro 3") (footprint "")
     )
+    (path "/f47f7cdf-3580-439c-86a6-80f9e434af39/a9615f49-d75d-411f-a192-f8d447b1167f"
+      (reference "U?") (unit 1) (value "can1_transmitter") (footprint "")
+    )
     (path "/8ed858a8-e638-495c-b31c-77c4342d4bce/b3824f86-f835-4bfd-957d-e4aadb0be4e8"
       (reference "U?") (unit 1) (value "ODrive Pro 0") (footprint "")
@@
     (path "/f47f7cdf-3580-439c-86a6-80f9e434af39/bd272f74-5169-48aa-b1af-95e0b50f6ffa"
       (reference "U?") (unit 1) (value "hand_trajectory_planner") (footprint "")
-    )
-    (path "/f47f7cdf-3580-439c-86a6-80f9e434af39/c455769e-b745-442e-94c5-85f755cdc5b2"
-      (reference "U?") (unit 1) (value "CRC_calculator") (footprint "")
     )
     (path "/f47f7cdf-3580-439c-86a6-80f9e434af39/c5e3ccae-a45d-4f4c-8f25-e9c9b687cf81"
@@
       (reference "U?") (unit 1) (value "50W, 2Ω Brake Resistor") (footprint "")
     )
-    (path "/f47f7cdf-3580-439c-86a6-80f9e434af39/f2ca9f06-88e8-42cc-a39c-22b7c0813816"
-      (reference "U?") (unit 1) (value "throw_scheduler") (footprint "")
-    )
     (path "/8ed858a8-e638-495c-b31c-77c4342d4bce/f2eeebc6-0e67-44f9-963a-7f2e6a51294e"
